File: Lesson 4/EE-Workshop.sch (EAGLE design)
At the start: 1 part

Commit message: Update EE-Workshop.sch
Parts:
- added C1, C2: .1UF, rcl:C-USC0805
- added IC1: NE555D, linear:NE555D
- added R1: 3K, rcl:R-US_R0805
- added R10: 6.2K, rcl:R-US_R0805
- added R11, R6: 1K, rcl:R-US_R0805
- added R2: 1.5K, rcl:R-US_R0805
- added R3: 1.3K, rcl:R-US_R0805
- added R4: (no value), rcl:R-US_R0805
- added R5: 1.1K, rcl:R-US_R0805
- added R7: 910, rcl:R-US_R0805
- added R8: 390, rcl:R-US_R0805
- added S1, S2, S3, S4, S5, S6, S7, S8: MOMENTARY-SWITCH-SPST-SMD-6.2MM-TALL, SparkFun-Switches:MOMENTARY-SWITCH-SPST-SMD-6.2MM-TALL
- added SG1: F/HMB, buzzer:F/HMB
- added T1: (no value), transistor:BCW60-NPN-SOT23-BEC
Connections:
- new net 0: BATT.-, C1.2, C2.2, IC1.GND, T1.E
- new net N$1: C2.1, IC1.CV
- new net N$10: SG1.-, T1.C
- new net N$5: IC1.Q, R1.1
- new net N$9: R1.2, T1.B
- new net TR: C1.1, IC1.THR, IC1.TR, S1.1, S2.1, S3.1, S4.1, S5.1, S6.1, S7.1, S8.1
- new net VCC: BATT.+, IC1.DIS, IC1.R, IC1.V+, R10.1, R10.2, R11.1, R11.2, R2.1, R2.2, R3.1, R3.2, R4.1, R4.2, R5.1, R5.2, R6.1, R6.2, R7.1, R7.2, R8.1, R8.2, S1.2, S2.2, S3.2, S4.2, S5.2, S6.2, S7.2, S8.2, SG1.+
